File: pcb/lt6c-pcb.kicad_pcb (KiCad board)
At the start: 2 copper layers, 62 x 66.4 mm, 19 parts, among them SW1 SW_Push, SW2 SW_Push, SW3 SW_Push, SW4 SW_Push, SW5 SW_Push, SW6 SW_Push, U1 XIAO-RP2040, U2 TPS76318, U3 PMW3360DM-T2QU

Commit message: Update LKBD libraries (#14)
Parts:
- U1: footprint LKBD_MCU:MCU_XIAO-RP2040 -> LKBD_MCU:MCU_XIAO_RP2040
- moved U3 8.70 mm to (148.2, 106.3)
Other:
- board text added: "XIAO RP2040"
