File: pcb/lt6c-pcb.kicad_sch (KiCad schematic)
At the start: 19 parts, among them SW1 SW_Push, SW2 SW_Push, SW3 SW_Push, SW4 SW_Push, SW5 SW_Push, SW6 SW_Push, U1 XIAO-RP2040, U2 TPS76318, U3 PMW3360DM-T2QU

Commit message: Update LKBD libraries (#14)
Parts:
- U1: footprint LKBD_MCU:MCU_XIAO-RP2040 -> LKBD_MCU:MCU_XIAO_RP2040
Changed lines of the file:
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@@
 		(at 153.67 19.05 270)
 		(unit 1)
-		(exclude_from_sim yes)
+		(exclude_from_sim no)
 		(in_bom no)
 		(on_board yes)
@@
 		(fields_autoplaced yes)
 		(property "Reference" "H1"
-			(at 158.115 17.7799 90)
+			(at 157.48 17.7799 90)
 			(effects
 				(font
@@
 		)
 		(property "Value" "MountingHole_Pad"
-			(at 158.115 20.3199 90)
+			(at 157.48 20.3199 90)
 			(effects
 				(font
@@
 			)
 		)
-		(property "Footprint" "LKBD_MCU:MCU_XIAO-RP2040"
+		(property "Footprint" "LKBD_MCU:MCU_XIAO_RP2040"
 			(at 47.244 50.292 0)
 			(effects
@@
 		(at 153.67 26.67 270)
 		(unit 1)
-		(exclude_from_sim yes)
+		(exclude_from_sim no)
 		(in_bom no)
 		(on_board yes)
@@
 		(fields_autoplaced yes)
 		(property "Reference" "H2"
-			(at 158.115 25.3999 90)
+			(at 157.48 25.3999 90)
 			(effects
 				(font
@@
 		)
 		(property "Value" "MountingHole_Pad"
-			(at 158.115 27.9399 90)
+			(at 157.48 27.9399 90)
 			(effects
 				(font
@@
 		(at 153.67 41.91 270)
 		(unit 1)
-		(exclude_from_sim yes)
+		(exclude_from_sim no)
 		(in_bom no)
 		(on_board yes)
@@
 		(fields_autoplaced yes)
 		(property "Reference" "H4"
-			(at 158.115 40.6399 90)
+			(at 157.48 40.6399 90)
 			(effects
 				(font
@@
 		)
 		(property "Value" "MountingHole_Pad"
-			(at 158.115 43.1799 90)
+			(at 157.48 43.1799 90)
 			(effects
 				(font
@@
 		(at 153.67 34.29 270)
 		(unit 1)
-		(exclude_from_sim yes)
+		(exclude_from_sim no)
 		(in_bom no)
 		(on_board yes)
@@
 		(fields_autoplaced yes)
 		(property "Reference" "H3"
-			(at 158.115 33.0199 90)
+			(at 157.48 33.0199 90)
 			(effects
 				(font
@@
 		)
 		(property "Value" "MountingHole_Pad"
-			(at 158.115 35.5599 90)
-			(effects
-				(font
+			(at 157.48 35.5599 90)
+			(effects
+				(font
